Commit message: Add affordance-aware dual-arm handover system
Extends the base UR3 dual-arm simulation with a semantic-guided
handover pipeline: OWL-v2 + SAM segmentation, Gemini-based grasp
region reasoning, AnyGrasp candidate generation, FoundationPose
pose completion, and a custom Affordance GT metric that measures
(from real Gazebo ground truth, invisible to the running system)
whether the object's functional end lands correctly in the
receiving hand. Includes ablation-study tooling and results
comparing the full semantic pipeline against a no-llm baseline
across four objects.

File: ur_gripper_gazebo/urdf/ur_gripper_hande.xacro (robot description, xacro)
@@ -1,170 +1,36 @@
 <?xml version="1.0"?>
 <robot xmlns:xacro="http://wiki.ros.org/xacro" name="ur_robot_gazebo">
-  <!--
-    This is a top-level xacro instantiating the Gazebo-specific version of the
-    'ur_robot' macro (ie: 'ur_robot_gazebo') and passing it values for all its
-    required arguments.
-    This file should be considered the Gazebo-specific variant of the file
-    with the same name in the ur_description package. It accepts the same
-    arguments, but instead of configuring everything for a real robot, will
-    generate a Gazebo-compatible URDF with a ros_control hardware_interface
-    attached to it.
-    Only use this top-level xacro if you plan on spawning the robot in Gazebo
-    'by itself', without any gripper or any other geometry attached.
-    If you need to attach an end-effector, camera or need to integrate the
-    robot into a larger workcell and want to spawn that as a single entity in
-    Gazebo, DO NOT EDIT THIS FILE.
-    Instead: create a new top-level xacro, give it a proper name, include the
-    required '.xacro' files, instantiate the models (ie: call the macros) and
-    connect everything by adding the appropriate joints.
-  -->
-  <!--
-    Import main macro.
-    NOTE: this imports the Gazebo-wrapper main macro, NOT the regular
-          xacro macro (which is hosted by ur_description).
-  -->
-  <xacro:include filename="$(find ur_gazebo)/urdf/ur_macro.xacro"/>
-  <!--Declare arguments -->
-  <xacro:arg name="joint_limit_params" default=""/>
-  <xacro:arg name="physical_params" default=""/>
-  <xacro:arg name="kinematics_params" default=""/>
-  <xacro:arg name="visual_params" default=""/>
-  <!--
-    legal values:
-      - hardware_interface/PositionJointInterface
-      - hardware_interface/VelocityJointInterface
-      - hardware_interface/EffortJointInterface
-    NOTE: this value must correspond to the controller configured in the
-          controller .yaml files in the 'config' directory.
-  -->
-  <xacro:arg name="transmission_hw_interface" default="hardware_interface/PositionJointInterface"/>
-  <xacro:arg name="safety_limits" default="false"/>
-  <xacro:arg name="safety_pos_margin" default="0.15"/>
-  <xacro:arg name="safety_k_position" default="20"/>
-  <!-- Instantiate the Gazebo robot and pass it all the required arguments. -->
-  <xacro:ur_robot_gazebo
-    prefix=""
-    joint_limits_parameters_file="$(arg joint_limit_params)"
-    kinematics_parameters_file="$(arg kinematics_params)"
-    physical_parameters_file="$(arg physical_params)"
-    visual_parameters_file="$(arg visual_params)"
-    transmission_hw_interface="$(arg transmission_hw_interface)"
-    safety_limits="$(arg safety_limits)"
-    safety_pos_margin="$(arg safety_pos_margin)"
-    safety_k_position="$(arg safety_k_position)"
-  />
-  <!--
-    Attach the Gazebo model to Gazebo's world frame.
-    Note: if you're looking to integrate a UR into a larger scene and need
-    to add EEFs or other parts, DO NOT change this file or the 'world' link
-    here. Create a NEW xacro instead and decide whether you need to add
-    a 'world' link there.
-  -->
-  <link name="world"/>
-  <joint name="world_joint" type="fixed">
-    <parent link="world"/>
-    <child link="base_link"/>
-    <origin xyz="0 0 0" rpy="0 0 0"/>
-  </joint>
-  <!-- Gripper -->
-  <xacro:arg name="grasp_plugin" default="false" />
-  <xacro:include filename="$(find robotiq_description)/urdf/robotiq_hande_gripper.urdf.xacro" />
-  <!-- Robotiq Coupler -->
-  <!--  + Height added by the coupler: 8mm -->
-  <!--  + Reference frame: at the middle (4mm) -->
-  <link name="robotiq_coupler">
-    <visual>
-      <geometry>
-        <mesh filename="package://robotiq_description/meshes/robotiq_85_coupler.stl" />
-      </geometry>
-      <material name="flat_black">
-        <color rgba="0 0 0 1.0"/>
-      </material>
-    </visual>
-    <collision>
-      <geometry>
-        <mesh filename="package://robotiq_description/meshes/robotiq_85_coupler.stl" />
-      </geometry>
-    </collision>
-    <inertial>
-      <origin xyz="2.073e-05   1.45286e-03  -1.1049e-03" rpy="0 0 0" />
-      <mass value="0.168" />
-      <inertia ixx="6.69695624e-05" ixy="5.21511788e-09" ixz="-2.74383009e-08"
-               iyy="7.85088161e-05" iyz="5.41105193e-07" izz="1.41819717e-04"/>
-    </inertial>
-  </link>
-  <joint name="robotiq_coupler_joint" type="fixed">
-    <origin xyz="0 0 0.004" rpy="0 0 ${-pi/2.0}" />
-    <parent link="tool0"/>
-    <child link="robotiq_coupler"/>
-  </joint>
-  <gazebo reference="robotiq_coupler">
-    <mu1>0.9</mu1>
-    <mu2>0.9</mu2>
-    <material>Gazebo/FlatBlack</material>
-  </gazebo>
-  <!-- Equivalent to the OpenRAVE manipulator denso_robotiq_hande_gripper -->
-  <link name="gripper_tip_link" />
-  <joint name="manipulator_dummy_joint" type="fixed">
-    <origin xyz="0 0 0.1441" rpy="0 0 0" />
-    <parent link="robotiq_coupler"/>
-    <child link="gripper_tip_link"/>
-  </joint>
-  <!-- Attach the robotiq hand-e gripper -->
-  <xacro:robotiq_hande_gripper prefix="" parent="robotiq_coupler" >
-    <origin xyz="0 0 0.004" rpy="0 0 ${-pi/2}"/>
-  </xacro:robotiq_hande_gripper>
-  <!-- Gazebo Force/Torque sensor plugin -->
-  <gazebo reference="wrist_3_joint">
-    <provideFeedback>true</provideFeedback>
-  </gazebo>
-  <!-- <gazebo reference="wrist_3_joint">
-    <preserveFixedJoint>true</preserveFixedJoint>
-  </gazebo> -->
-  <gazebo>
-    <plugin name="ft_sensor" filename="libgazebo_ros_ft_sensor.so">
-      <updateRate>500.0</updateRate>
-      <topicName>wrench</topicName>
-      <gaussianNoise>0.0</gaussianNoise>
-      <jointName>wrist_3_joint</jointName>
-    </plugin>
-  </gazebo>
-  <!-- Gazebo grasping plugin
-      grasp_plugin True = custom gazebo_grasp_fix
-      grasp_plugin False = gazebo_gripper
-  -->
-  <xacro:if value="$(arg grasp_plugin)">
-    <gazebo>
-      <plugin name="gazebo_grasp_fix" filename="libgazebo_grasp_fix.so">
-            <arm>
-              <arm_name>robotiq_hande</arm_name>
-              <palm_link>wrist_3_link</palm_link>
-              <gripper_link>hande_right_finger</gripper_link>
-              <gripper_link>hande_left_finger</gripper_link>
-            </arm>
-          <forces_angle_tolerance>100</forces_angle_tolerance>
-          <update_rate>100</update_rate>
-          <grip_count_threshold>5</grip_count_threshold>
-          <max_grip_count>30</max_grip_count>
-          <release_tolerance>0.0015</release_tolerance>
-          <disable_collisions_on_attach>false</disable_collisions_on_attach>
-          <contact_topic>__default_topic__</contact_topic>
-        </plugin>
-    </gazebo>
-  </xacro:if>
-  <xacro:unless value="$(arg grasp_plugin)">
-    <gazebo>
-      <gripper name="gazebo_gripper">
-        <grasp_check>
-          <attach_steps>2</attach_steps>
-          <detach_steps>2</detach_steps>
-          <min_contact_count>3</min_contact_count>
-        </grasp_check>
-        <gripper_link>hande_right_finger</gripper_link>
-        <gripper_link>hande_left_finger</gripper_link>
-        <palm_link>wrist_3_link</palm_link>
-      </gripper>
-    </gazebo>
-  </xacro:unless>
-  <!-- Gazebo grasping plugin -->
+  <xacro:macro name="ur_gripper_hande" params="
+    prefix
+    ft_prefix
+    parent
+    *origin
+    joint_limits_parameters_file
+    kinematics_parameters_file
+    physical_parameters_file
+    visual_parameters_file
+    transmission_hw_interface:=hardware_interface/PositionJointInterface
+    safety_limits:=false safety_pos_margin:=0.15 safety_k_position:=20">
+  <xacro:include filename="$(find ur_gripper_gazebo)/urdf/ur_macro.xacro"/>
+    <!-- Instantiate the Gazebo robot and pass it all the required arguments. -->
+    <xacro:ur_robot_gazebo
+      prefix="${prefix}"
+      joint_limits_parameters_file="${joint_limits_parameters_file}"
+      kinematics_parameters_file="${kinematics_parameters_file}"
+      physical_parameters_file="${physical_parameters_file}"
+      visual_parameters_file="${visual_parameters_file}"
+      transmission_hw_interface="${transmission_hw_interface}"
+      safety_limits="${safety_limits}"
+      safety_pos_margin="${safety_pos_margin}"
+      safety_k_position="${safety_k_position}"
+    />
+    <joint name="${prefix}${parent}_joint" type="fixed">
+      <parent link="${parent}"/>
+      <child link="${prefix}base_link"/>
+      <xacro:insert_block name="origin"/>
+    </joint>
+    <!-- Gripper -->
+    <xacro:include filename="$(find ur_gripper_description)/urdf/robotiq_hande_gripper_manual_exchanger.urdf.xacro" />
+    <xacro:robotiq_hande_gripper_adapter_manual_exchanger prefix="${prefix}" parent="${prefix}tool0" ft_prefix="${ft_prefix}"/>
+  </xacro:macro>
 </robot>
